Commit message: Added Localization

File: estimation_mapping/urdf/simple.urdf (robot description, URDF)
Before this commit: robot deepracer_simple, 2 links, 1 joints
Links:
- added link front_left_wheel, mass 0.1; collision cylinder length=0.03 radius=0.04; visual cylinder length=0.03 radius=0.04
- added link front_right_wheel, mass 0.1; collision cylinder length=0.03 radius=0.04; visual cylinder length=0.03 radius=0.04
- added link rear_left_wheel, mass 0.1; collision cylinder length=0.03 radius=0.04; visual cylinder length=0.03 radius=0.04
- added link rear_right_wheel, mass 0.1; collision cylinder length=0.03 radius=0.04; visual cylinder length=0.03 radius=0.04
- link base_link: mass 1.0 -> 1.5; geometry collision box size=0.32 0.20 0.08; visual box size=0.32 0.20 0.08
- link laser: geometry visual cylinder length=0.04 radius=0.03
Joints:
- added joint front_left_wheel_joint: type fixed, parent base_link, child front_left_wheel, origin xyz=0.12 0.115 0.04 rpy=0 0 0
- added joint front_right_wheel_joint: type fixed, parent base_link, child front_right_wheel, origin xyz=0.12 -0.115 0.04 rpy=0 0 0
- added joint rear_left_wheel_joint: type fixed, parent base_link, child rear_left_wheel, origin xyz=-0.12 0.115 0.04 rpy=0 0 0
- added joint rear_right_wheel_joint: type fixed, parent base_link, child rear_right_wheel, origin xyz=-0.12 -0.115 0.04 rpy=0 0 0
